File: snowman.sch (KiCad schematic (older format))
At the start: 8 parts, among them SW1 SW_SPST, SW2 SW_SPST, SW3 SW_SPST, U1 ATTINY85-20SU

Commit message: Update Footprints
Update piezo buzzer footprint, making it wider for easier hand soldering.
Update button schematic to change pin 2 to pin 4 to match buttons being used
Update LED footprint in schematic to 3mm
Parts:
- D1: footprint LEDs:LED_D5.0mm -> LEDs:LED_D3.0mm
- SW1, SW2, SW3: symbol SW_SPST -> SW_SPST4
Connections:
- net GND: now also SW1.4 (B), SW2.4 (B), SW3.4 (B); no longer SW1.2 (B), SW2.2 (B), SW3.2 (B)
Changed lines of the file:
@@
 LIBS:switches
 LIBS:piezo
+LIBS:sw_spst
 LIBS:snowman-cache
 EELAYER 26 0
@@
 F 0 "D1" H 5531 1964 50  0000 C CNN
 F 1 "LED" H 5531 2055 50  0000 C CNN
-F 2 "LEDs:LED_D5.0mm" H 5539 2219 50  0001 C CNN
+F 2 "LEDs:LED_D3.0mm" H 5539 2219 50  0001 C CNN
 F 3 "" H 5539 2219 50  0001 C CNN
 	1    5539 2219
@@
 $EndComp
 $Comp
-L SW_SPST SW2
+L SW_SPST4 SW2
 U 1 1 59380E68
 P 6107 3447
@@
 $EndComp
 $Comp
-L SW_SPST SW1
+L SW_SPST4 SW1
 U 1 1 59380F18
 P 6149 2941
@@
 $EndComp
 $Comp
-L SW_SPST SW3
+L SW_SPST4 SW3
 U 1 1 59380F75
 P 6059 3937

Commit message: Add DigiKey Product ID
Add DigiKey product id's to all parts for creating BOM file
Add price spreadsheet
Parts:
- BT1: DigiKey (none) -> 36-3002CT-ND
- D1: DigiKey (none) -> 846-1190-ND
- PIEZO1: DigiKey (none) -> 490-4683-1-ND
- R1: DigiKey (none) -> 311-100HRCT-ND
- SW1, SW2, SW3: DigiKey (none) -> CKN9104CT-ND
- U1: DigiKey (none) -> ATTINY85-20SU-ND
Changed lines of the file:
@@
 F 2 "Battery_Holders:Keystone_3002_1x2032-CoinCell" V 1280 2543 50  0001 C CNN
 F 3 "" V 1280 2543 50  0001 C CNN
+F 4 "36-3002CT-ND" H 1280 2483 60  0001 C CNN "DigiKey"
 	1    1280 2483
 	1    0    0    -1
@@
 F 2 "ATTiny85:ATTiny85-20SU" H 4989 2469 50  0001 C CIN
 F 3 "" H 4039 2469 50  0001 C CNN
+F 4 "ATTINY85-20SU-ND" H 4039 2469 60  0001 C CNN "DigiKey"
 	1    4039 2469
 	-1   0    0    -1
@@
 F 2 "LEDs:LED_D3.0mm" H 5539 2219 50  0001 C CNN
 F 3 "" H 5539 2219 50  0001 C CNN
+F 4 "846-1190-ND" H 5539 2219 60  0001 C CNN "DigiKey"
 	1    5539 2219
 	-1   0    0    1
@@
 F 2 "Buttons:Button_SMD-PTS525SM15SMTR2-LFS" H 6107 3447 50  0001 C CNN
 F 3 "" H 6107 3447 50  0001 C CNN
+F 4 "CKN9104CT-ND" H 6107 3447 60  0001 C CNN "DigiKey"
 	1    6107 3447
 	1    0    0    -1
@@
 F 2 "Buttons:Button_SMD-PTS525SM15SMTR2-LFS" H 6149 2941 50  0001 C CNN
 F 3 "" H 6149 2941 50  0001 C CNN
+F 4 "CKN9104CT-ND" H 6149 2941 60  0001 C CNN "DigiKey"
 	1    6149 2941
 	1    0    0    -1
@@
 F 2 "Buttons:Button_SMD-PTS525SM15SMTR2-LFS" H 6059 3937 50  0001 C CNN
 F 3 "" H 6059 3937 50  0001 C CNN
+F 4 "CKN9104CT-ND" H 6059 3937 60  0001 C CNN "DigiKey"
 	1    6059 3937
 	1    0    0    -1
@@
 F 2 "Resistors_SMD:R_0603_HandSoldering" V 5769 2219 50  0001 C CNN
 F 3 "" H 5839 2219 50  0001 C CNN
+F 4 "311-100HRCT-ND" V 5839 2219 60  0001 C CNN "DigiKey"
 	1    5839 2219
 	0    1    1    0
@@
 F 2 "Piezo:Piezo-PKMCS0909E4000-R1" H 6077 2319 60  0001 C CNN
 F 3 "" H 6077 2319 60  0000 C CNN
+F 4 "490-4683-1-ND" H 6077 2319 60  0001 C CNN "DigiKey"
 	1    6077 2319
 	0    1    1    0

Commit message: KiCad Symbol Update
Update to how KiCad uses symbols
Parts:
- BT1: symbol Battery_Cell -> device:Battery_Cell
- D1: symbol LED -> device:LED
- PIEZO1: symbol PIEZO -> piezo:PIEZO
- R1: symbol R -> device:R
- SW1, SW2, SW3: symbol SW_SPST4 -> sw_spst:SW_SPST4
- U1: symbol ATTINY85-20SU -> atmel:ATTINY85-20SU
Changed lines of the file:
@@
-EESchema Schematic File Version 2
-LIBS:power
-LIBS:device
-LIBS:transistors
-LIBS:conn
-LIBS:linear
-LIBS:regul
-LIBS:74xx
-LIBS:cmos4000
-LIBS:adc-dac
-LIBS:memory
-LIBS:xilinx
-LIBS:microcontrollers
-LIBS:dsp
-LIBS:microchip
-LIBS:analog_switches
-LIBS:motorola
-LIBS:texas
-LIBS:intel
-LIBS:audio
-LIBS:interface
-LIBS:digital-audio
-LIBS:philips
-LIBS:display
-LIBS:cypress
-LIBS:siliconi
-LIBS:opto
-LIBS:atmel
-LIBS:contrib
-LIBS:valves
-LIBS:switches
-LIBS:piezo
-LIBS:sw_spst
+EESchema Schematic File Version 4
 LIBS:snowman-cache
 EELAYER 26 0
@@
 $EndDescr
 $Comp
-L Battery_Cell BT1
+L device:Battery_Cell BT1
 U 1 1 593808F0
 P 1280 2483
@@
 $EndComp
 $Comp
-L ATTINY85-20SU U1
+L atmel:ATTINY85-20SU U1
 U 1 1 59380980
 P 4039 2469
@@
 $EndComp
 $Comp
-L LED D1
+L device:LED D1
 U 1 1 59380BF5
 P 5539 2219
@@
 $EndComp
 $Comp
-L SW_SPST4 SW2
+L sw_spst:SW_SPST4 SW2
 U 1 1 59380E68
 P 6107 3447
@@
 $EndComp
 $Comp
-L SW_SPST4 SW1
+L sw_spst:SW_SPST4 SW1
 U 1 1 59380F18
 P 6149 2941
@@
 $EndComp
 $Comp
-L SW_SPST4 SW3
+L sw_spst:SW_SPST4 SW3
 U 1 1 59380F75
 P 6059 3937
@@
 $EndComp
 $Comp
-L R R1
+L device:R R1
 U 1 1 59381195
 P 5839 2219
@@
 VCC
 $Comp
-L PIEZO PIEZO1
+L piezo:PIEZO PIEZO1
 U 1 1 59382115
 P 6077 2319
@@
 $EndComp
 $Comp
-L GND #PWR01
+L power:GND #PWR01
 U 1 1 59384465
 P 1280 2719
@@
 $EndComp
 $Comp
-L GND #PWR02
+L power:GND #PWR02
 U 1 1 593844F3
 P 2689 2719
@@
 $EndComp
 $Comp
-L GND #PWR03
+L power:GND #PWR03
 U 1 1 593845ED
 P 6059 2219
@@
 $EndComp
 $Comp
-L GND #PWR04
+L power:GND #PWR04
 U 1 1 59384742
 P 6297 2319
@@
 $EndComp
 $Comp
-L GND #PWR05
+L power:GND #PWR05
 U 1 1 5938480F
 P 6431 2941
@@
 $EndComp
 $Comp
-L GND #PWR06
+L power:GND #PWR06
 U 1 1 593848CA
 P 6398 3447
@@
 $EndComp
 $Comp
-L GND #PWR07
+L power:GND #PWR07
 U 1 1 59384973
 P 6344 3937
